File: teensy-oled-badge.sch (KiCad schematic (older format))
At the start: 6 parts, among them J1 TEENSY-LC, J2 OLED_128x64

Commit message: initial draft of layout
Parts:
- removed CAP?: CAPSENSE_CIRCLE, symbol CAPSENSE_CIRCLE
- CAP1, CAP2, CAP3: renamed from CAP?; footprint (none) -> Wickerlib:CAPSENSE_CIRCLE_D10
Connections:
- no-connect marks 1 -> 24
Changed lines of the file:
@@
 NoConn ~ 7425 3000
 $Comp
-L CAPSENSE_CIRCLE CAP?
+L CAPSENSE_CIRCLE CAP1
 U 1 1 57E17B23
 P 6650 4125
-F 0 "CAP?" H 6900 4225 60  0000 L CNN
+F 0 "CAP1" H 6900 4225 60  0000 L CNN
 F 1 "CAPSENSE_CIRCLE" H 6900 4025 60  0000 L CNN
-F 2 "" H 6650 4125 60  0000 C CNN
+F 2 "Wickerlib:CAPSENSE_CIRCLE_D10" H 6650 4125 60  0001 C CNN
 F 3 "" H 6650 4125 60  0000 C CNN
 	1    6650 4125
@@
 $EndComp
 $Comp
-L CAPSENSE_CIRCLE CAP?
+L CAPSENSE_CIRCLE CAP2
 U 1 1 57E17C95
 P 6700 4600
-F 0 "CAP?" H 6950 4700 60  0000 L CNN
+F 0 "CAP2" H 6950 4700 60  0000 L CNN
 F 1 "CAPSENSE_CIRCLE" H 6950 4500 60  0000 L CNN
-F 2 "" H 6700 4600 60  0000 C CNN
+F 2 "Wickerlib:CAPSENSE_CIRCLE_D10" H 6700 4600 60  0001 C CNN
 F 3 "" H 6700 4600 60  0000 C CNN
 	1    6700 4600
@@
 $EndComp
 $Comp
-L CAPSENSE_CIRCLE CAP?
+L CAPSENSE_CIRCLE CAP3
 U 1 1 57E17E3A
 P 6950 1675
-F 0 "CAP?" H 7200 1775 60  0000 L CNN
+F 0 "CAP3" H 7200 1775 60  0000 L CNN
 F 1 "CAPSENSE_CIRCLE" H 7200 1575 60  0000 L CNN
-F 2 "" H 6950 1675 60  0000 C CNN
+F 2 "Wickerlib:CAPSENSE_CIRCLE_D10" H 6950 1675 60  0001 C CNN
 F 3 "" H 6950 1675 60  0000 C CNN
 	1    6950 1675
-	1    0    0    -1
-$EndComp
-$Comp
-L CAPSENSE_CIRCLE CAP?
-U 1 1 57E180FB
-P 6975 1150
-F 0 "CAP?" H 7225 1250 60  0000 L CNN
-F 1 "CAPSENSE_CIRCLE" H 7225 1050 60  0000 L CNN
-F 2 "" H 6975 1150 60  0000 C CNN
-F 3 "" H 6975 1150 60  0000 C CNN
-	1    6975 1150
 	1    0    0    -1
 $EndComp
@@
 	5475 2650 5600 2650
 Wire Wire Line
-	5600 2650 5600 1150
-Wire Wire Line
-	5600 1150 6625 1150
-Wire Wire Line
 	5475 2750 5675 2750
 Wire Wire Line
@@
 Wire Wire Line
 	5675 1675 6600 1675
+NoConn ~ 5475 2350
+NoConn ~ 5525 2050
+NoConn ~ 5525 1950
+NoConn ~ 5475 2450
+NoConn ~ 5475 2550
+NoConn ~ 5475 2850
+NoConn ~ 5475 2950
+NoConn ~ 5475 3050
+NoConn ~ 5475 3150
+NoConn ~ 5475 3750
+NoConn ~ 5475 3850
+NoConn ~ 5475 3950
+NoConn ~ 5475 4050
+NoConn ~ 5475 4150
+NoConn ~ 5475 4250
+NoConn ~ 5475 4350
+NoConn ~ 5475 4450
+NoConn ~ 5525 4800
+NoConn ~ 5525 4900
+NoConn ~ 5525 5000
+NoConn ~ 5475 5250
+NoConn ~ 5475 5350
+NoConn ~ 5600 2650
 $EndSCHEMATC
