File: teensy-oled-badge.kicad_pcb (KiCad board)
At the start: 2 copper layers, 32.6 x 41.2 mm, 7 parts, among them J1 TEENSY-LC, J2 OLED_128x64

Commit message: initial draft of layout
Parts:
- removed the G*** at (161.9, 127.4)
- added CAP1: CAPSENSE_CIRCLE, Wickerlib:CAPSENSE_CIRCLE_D10, F.Cu at (128.6, 98.9)
- added CAP2: CAPSENSE_CIRCLE, Wickerlib:CAPSENSE_CIRCLE_D10, F.Cu at (128.6, 111.3)
- added CAP3: CAPSENSE_CIRCLE, Wickerlib:CAPSENSE_CIRCLE_D10, F.Cu at (128.6, 123.5)
- REF**: moved to B.Cu
- moved REF** 38.8 mm to (128.5, 111.5), turned to 90 degrees
- moved G*** 9.37 mm to (146.4, 109.6)
- moved J2 1.77 mm to (164.1, 102.9)
Routing:
- net /CS: track 32.1 -> 67.6 mm, vias 1 -> 3
- net /DC: track 28.9 -> 60.7 mm, vias 1 -> 3
- net /Data: track 25.2 -> 55.6 mm, vias 0 -> 1
- net /CLK: track 26.8 -> 56.8 mm, vias 1 -> 3
- net Net-(CAP2-Pad1): track 0.00 -> 28.6 mm, vias 0 -> 2
- net Net-(CAP1-Pad1): track 0.00 -> 27.6 mm, vias 0 -> 1
- net /VIN: track 0.00 -> 25.4 mm
- net /RST: track 19.9 -> 40.1 mm, vias 0 -> 1
- net Net-(CAP3-Pad1): track 0.00 -> 20.0 mm
- added copper zone on B.Cu, net /GND
- removed copper zone on B.Cu, net /VIN
Other:
- board size 32.6 x 41.2 mm -> 68.7 x 41.2 mm
- board text added: "A"
- board text added: "B"
- board text added: "C"

Commit message: fix DRC errors
Parts:
- removed G***: LOGO, teensy-big-oled:osh-park-logo-300dpi-normal-copper
- removed G***: LOGO, teensy-big-oled:osh-park-logo-300dpi-normal-silk
- moved CAP3 1.99 mm to (127.9, 125.3)
- moved CAP1 1.39 mm to (127.4, 98.1)
- moved CAP2 1.00 mm to (127.6, 111.1)
Routing:
- net /CS: track 67.6 -> 33.1 mm, vias 3 -> 1
- net /DC: track 60.7 -> 29.9 mm, vias 3 -> 1
- net /CLK: track 56.8 -> 27.8 mm, vias 3 -> 1
- net /Data: track 55.6 -> 26.8 mm, vias 1 -> 0
- net /RST: track 40.1 -> 23.3 mm, vias 1 -> 0
- net /VIN: track 25.4 -> 12.9 mm
- net Net-(CAP3-Pad1): track 20.0 -> 23.7 mm
- net Net-(CAP1-Pad1): track 27.6 -> 29.0 mm
- net Net-(CAP2-Pad1): track 28.6 -> 29.5 mm
Other:
- net class Default: clearance 0.1524 -> 0.254; trace_width 0.254 -> 0.2286
- rule trace_clearance: 0.1524 -> 0.254
- rule trace_min: 0.254 -> 0.2286

Commit message: remove uneeded text
Parts:
- removed the REF** at (146.1, 103.5)
Changed lines of the file:
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@@
     (tracks 81)
     (zones 0)
-    (modules 7)
+    (modules 6)
     (nets 35)
   )
@@
     (34 B.Paste user)
     (35 F.Paste user)
-    (36 B.SilkS user hide)
+    (36 B.SilkS user)
     (37 F.SilkS user)
     (38 B.Mask user)
@@
   )
   (module Wickerlib:Symbol_OSHW-Logo_SilkScreen (layer B.Cu)
-    (at 146.05 103.505 90)
+    (at 128.4732 111.4552 90)
     (descr "Symbol, OSHW-Logo, Silk Screen,")
     (tags "Symbol, OSHW-Logo, Silk Screen,")
@@
       (effects (font (size 1 1) (thickness 0.15)) (justify mirror))
     )
-    (fp_text value Symbol_OSHW-Logo_SilkScreen (at 0.30988 -6.56082 90) (layer B.Fab)
+    (fp_text value Symbol_OSHW-Logo_SilkScreen (at 0.30988 -6.56082 90) (layer B.Fab) hide
       (effects (font (size 1 1) (thickness 0.15)) (justify mirror))
     )
@@
     (fp_line (start 0.35052 -0.89916) (end 0.7493 -1.89992) (layer B.SilkS) (width 0.15))
   )
-  (module Wickerlib:Symbol_OSHW-Logo_SilkScreen (layer B.Cu)
-    (at 128.4732 111.4552 90)
-    (descr "Symbol, OSHW-Logo, Silk Screen,")
-    (tags "Symbol, OSHW-Logo, Silk Screen,")
-    (fp_text reference REF** (at 0.09906 4.38912 90) (layer B.SilkS) hide
-      (effects (font (size 1 1) (thickness 0.15)) (justify mirror))
-    )
-    (fp_text value Symbol_OSHW-Logo_SilkScreen (at 0.30988 -6.56082 90) (layer B.Fab) hide
-      (effects (font (size 1 1) (thickness 0.15)) (justify mirror))
-    )
-    (fp_line (start 1.66878 -2.68986) (end 2.02946 -4.16052) (layer B.SilkS) (width 0.15))
-    (fp_line (start 2.02946 -4.16052) (end 2.30886 -3.0988) (layer B.SilkS) (width 0.15))
-    (fp_line (start 2.30886 -3.0988) (end 2.61874 -4.17068) (layer B.SilkS) (width 0.15))
-    (fp_line (start 2.61874 -4.17068) (end 2.9591 -2.72034) (layer B.SilkS) (width 0.15))
-    (fp_line (start 0.24892 -3.38074) (end 1.03886 -3.37058) (layer B.SilkS) (width 0.15))
-    (fp_line (start 1.03886 -3.37058) (end 1.04902 -3.38074) (layer B.SilkS) (width 0.15))
-    (fp_line (start 1.04902 -3.38074) (end 1.04902 -3.37058) (layer B.SilkS) (width 0.15))
-    (fp_line (start 1.08966 -2.65938) (end 1.08966 -4.20116) (layer B.SilkS) (width 0.15))
-    (fp_line (start 0.20066 -2.64922) (end 0.20066 -4.21894) (layer B.SilkS) (width 0.15))
-    (fp_line (start 0.20066 -4.21894) (end 0.21082 -4.20878) (layer B.SilkS) (width 0.15))
-    (fp_line (start -0.35052 -2.75082) (end -0.70104 -2.66954) (layer B.SilkS) (width 0.15))
-    (fp_line (start -0.70104 -2.66954) (end -1.02108 -2.65938) (layer B.SilkS) (width 0.15))
-    (fp_line (start -1.02108 -2.65938) (end -1.25984 -2.86004) (layer B.SilkS) (width 0.15))
-    (fp_line (start -1.25984 -2.86004) (end -1.29032 -3.12928) (layer B.SilkS) (width 0.15))
-    (fp_line (start -1.29032 -3.12928) (end -1.04902 -3.37058) (layer B.SilkS) (width 0.15))
-    (fp_line (start -1.04902 -3.37058) (end -0.6604 -3.50012) (layer B.SilkS) (width 0.15))
-    (fp_line (start -0.6604 -3.50012) (end -0.48006 -3.66014) (layer B.SilkS) (width 0.15))
-    (fp_line (start -0.48006 -3.66014) (end -0.43942 -3.95986) (layer B.SilkS) (width 0.15))
-    (fp_line (start -0.43942 -3.95986) (end -0.67056 -4.18084) (layer B.SilkS) (width 0.15))
-    (fp_line (start -0.67056 -4.18084) (end -0.9906 -4.20878) (layer B.SilkS) (width 0.15))
-    (fp_line (start -0.9906 -4.20878) (end -1.34112 -4.09956) (layer B.SilkS) (width 0.15))
-    (fp_line (start -2.37998 -2.64922) (end -2.6289 -2.66954) (layer B.SilkS) (width 0.15))
-    (fp_line (start -2.6289 -2.66954) (end -2.8702 -2.91084) (layer B.SilkS) (width 0.15))
-    (fp_line (start -2.8702 -2.91084) (end -2.9591 -3.40106) (layer B.SilkS) (width 0.15))
-    (fp_line (start -2.9591 -3.40106) (end -2.93116 -3.74904) (layer B.SilkS) (width 0.15))
-    (fp_line (start -2.93116 -3.74904) (end -2.7305 -4.06908) (layer B.SilkS) (width 0.15))
-    (fp_line (start -2.7305 -4.06908) (end -2.47904 -4.191) (layer B.SilkS) (width 0.15))
-    (fp_line (start -2.47904 -4.191) (end -2.16916 -4.11988) (layer B.SilkS) (width 0.15))
-    (fp_line (start -2.16916 -4.11988) (end -1.95072 -3.93954) (layer B.SilkS) (width 0.15))
-    (fp_line (start -1.95072 -3.93954) (end -1.8796 -3.4798) (layer B.SilkS) (width 0.15))
-    (fp_line (start -1.8796 -3.4798) (end -1.9304 -3.07086) (layer B.SilkS) (width 0.15))
-    (fp_line (start -1.9304 -3.07086) (end -2.03962 -2.78892) (layer B.SilkS) (width 0.15))
-    (fp_line (start -2.03962 -2.78892) (end -2.4003 -2.65938) (layer B.SilkS) (width 0.15))
-    (fp_line (start -1.78054 -0.92964) (end -2.03962 -1.49098) (layer B.SilkS) (width 0.15))
-    (fp_line (start -2.03962 -1.49098) (end -1.50114 -2.00914) (layer B.SilkS) (width 0.15))
-    (fp_line (start -1.50114 -2.00914) (end -0.98044 -1.7399) (layer B.SilkS) (width 0.15))
-    (fp_line (start -0.98044 -1.7399) (end -0.70104 -1.89992) (layer B.SilkS) (width 0.15))
-    (fp_line (start 0.73914 -1.8796) (end 1.06934 -1.6891) (layer B.SilkS) (width 0.15))
-    (fp_line (start 1.06934 -1.6891) (end 1.50876 -2.0193) (layer B.SilkS) (width 0.15))
-    (fp_line (start 1.50876 -2.0193) (end 1.9812 -1.52908) (layer B.SilkS) (width 0.15))
-    (fp_line (start 1.9812 -1.52908) (end 1.69926 -1.04902) (layer B.SilkS) (width 0.15))
-    (fp_line (start 1.69926 -1.04902) (end 1.88976 -0.57912) (layer B.SilkS) (width 0.15))
-    (fp_line (start 1.88976 -0.57912) (end 2.49936 -0.39116) (layer B.SilkS) (width 0.15))
-    (fp_line (start 2.49936 -0.39116) (end 2.49936 0.28956) (layer B.SilkS) (width 0.15))
-    (fp_line (start 2.49936 0.28956) (end 1.94056 0.42926) (layer B.SilkS) (width 0.15))
-    (fp_line (start 1.94056 0.42926) (end 1.7399 1.00076) (layer B.SilkS) (width 0.15))
-    (fp_line (start 1.7399 1.00076) (end 2.00914 1.47066) (layer B.SilkS) (width 0.15))
-    (fp_line (start 2.00914 1.47066) (end 1.53924 1.9812) (layer B.SilkS) (width 0.15))
-    (fp_line (start 1.53924 1.9812) (end 1.02108 1.71958) (layer B.SilkS) (width 0.15))
-    (fp_line (start 1.02108 1.71958) (end 0.55118 1.92024) (layer B.SilkS) (width 0.15))
-    (fp_line (start 0.55118 1.92024) (end 0.381 2.46126) (layer B.SilkS) (width 0.15))
-    (fp_line (start 0.381 2.46126) (end -0.30988 2.47904) (layer B.SilkS) (width 0.15))
-    (fp_line (start -0.30988 2.47904) (end -0.5207 1.9304) (layer B.SilkS) (width 0.15))
-    (fp_line (start -0.5207 1.9304) (end -0.9398 1.76022) (layer B.SilkS) (width 0.15))
-    (fp_line (start -0.9398 1.76022) (end -1.49098 2.02946) (layer B.SilkS) (width 0.15))
-    (fp_line (start -1.49098 2.02946) (end -2.00914 1.50114) (layer B.SilkS) (width 0.15))
-    (fp_line (start -2.00914 1.50114) (end -1.76022 0.96012) (layer B.SilkS) (width 0.15))
-    (fp_line (start -1.76022 0.96012) (end -1.9304 0.48006) (layer B.SilkS) (width 0.15))
-    (fp_line (start -1.9304 0.48006) (end -2.47904 0.381) (layer B.SilkS) (width 0.15))
-    (fp_line (start -2.47904 0.381) (end -2.4892 -0.32004) (layer B.SilkS) (width 0.15))
-    (fp_line (start -2.4892 -0.32004) (end -1.9304 -0.5207) (layer B.SilkS) (width 0.15))
-    (fp_line (start -1.9304 -0.5207) (end -1.7907 -0.91948) (layer B.SilkS) (width 0.15))
-    (fp_line (start 0.35052 -0.89916) (end 0.65024 -0.7493) (layer B.SilkS) (width 0.15))
-    (fp_line (start 0.65024 -0.7493) (end 0.8509 -0.55118) (layer B.SilkS) (width 0.15))
-    (fp_line (start 0.8509 -0.55118) (end 1.00076 -0.14986) (layer B.SilkS) (width 0.15))
-    (fp_line (start 1.00076 -0.14986) (end 1.00076 0.24892) (layer B.SilkS) (width 0.15))
-    (fp_line (start 1.00076 0.24892) (end 0.8509 0.59944) (layer B.SilkS) (width 0.15))
-    (fp_line (start 0.8509 0.59944) (end 0.39878 0.94996) (layer B.SilkS) (width 0.15))
-    (fp_line (start 0.39878 0.94996) (end -0.0508 1.00076) (layer B.SilkS) (width 0.15))
-    (fp_line (start -0.0508 1.00076) (end -0.44958 0.89916) (layer B.SilkS) (width 0.15))
-    (fp_line (start -0.44958 0.89916) (end -0.8509 0.55118) (layer B.SilkS) (width 0.15))
-    (fp_line (start -0.8509 0.55118) (end -1.00076 0.09906) (layer B.SilkS) (width 0.15))
-    (fp_line (start -1.00076 0.09906) (end -0.94996 -0.39878) (layer B.SilkS) (width 0.15))
-    (fp_line (start -0.94996 -0.39878) (end -0.70104 -0.70104) (layer B.SilkS) (width 0.15))
-    (fp_line (start -0.70104 -0.70104) (end -0.35052 -0.89916) (layer B.SilkS) (width 0.15))
-    (fp_line (start -0.35052 -0.89916) (end -0.70104 -1.89992) (layer B.SilkS) (width 0.15))
-    (fp_line (start 0.35052 -0.89916) (end 0.7493 -1.89992) (layer B.SilkS) (width 0.15))
-  )
   (module Wickerlib:CAPSENSE_CIRCLE_D10 (layer F.Cu)
     (at 127.4318 98.0948 90)
@@
     (effects (font (size 1.5 1.5) (thickness 0.3)))
   )
-  (gr_text "DREW FUSTINI" (at 149.987 104.521 270) (layer B.Mask)
+  (gr_text "DREW FUSTINI" (at 159.0802 111.5314 270) (layer B.SilkS)
     (effects (font (size 1.5 1.5) (thickness 0.3)) (justify mirror))
   )
